File: machine-keeper.kicad_pcb (KiCad board)
At the start: 4 copper layers, 31.1 x 15.5 mm, 26 parts, among them J101 USB_B_Micro, U101 LIS2HH12, U102 TLV71333PDBV, U103 STM32F302K8Ux, U104 AT25DF041x-UxN-x, Y101 8MHz

Commit message: Work on schematic
Parts:
- added NT101: Net-Tie_2, NetTie:NetTie-2_SMD_Pad0.5mm, F.Cu at (67.9, 53.4)
- Y101: value 8MHz -> Crystal_GND24; footprint Crystal:Crystal_SMD_5032-2Pin_5.0x3.2mm -> Crystal:Crystal_SMD_3225-4Pin_3.2x2.5mm
- moved C102 2.03 mm to (87.3, 54.1)
- moved Y101 1.04 mm to (84.7, 53.0)
- moved U103 0.26 mm to (83.0, 59.0)
- turned C103 to 90 degrees
Connections:
- Y101 pad 2: Net-(C103-Pad1) -> GND
Routing:
- net Net-(C102-Pad1): track 6.88 -> 0.00 mm
- net Net-(C103-Pad1): track 5.35 -> 0.00 mm
- net /SWCLK: track 0.89 -> 0.00 mm, vias 1 -> 0
- net /SWDIO: track 0.85 -> 0.00 mm, vias 1 -> 0
- net /USB_DP: track 0.80 -> 0.00 mm, vias 1 -> 0
- net /USB_DM: track 0.78 -> 0.00 mm, vias 1 -> 0
