File: machine-keeper.sch (KiCad schematic (older format))
At the start: 8 parts

Commit message: Work on schematic
Parts:
- added U?: TLV71333PDBV, Package_TO_SOT_SMD:SOT-23-5, symbol Regulator_Linear:TLV71333PDBV
Connections:
- wire segments 13 -> 31
Other:
- note added: "TODO:\n- Add ideal diode part\n- Add battery holder\n- Remove net tie\n- Add TVS array part\n- Add LED part"
- note removed: "TODO:\n- Add ideal diode part\n- Add battery holder\n- Remove net tie"
Changed lines of the file:
@@
 U 1 1 5BA67CA8
 P 5750 4000
-F 0 "U?" H 5750 5078 50  0000 C CNN
-F 1 "STM32F302K8Ux" H 5750 4987 50  0000 C CNN
+F 0 "U?" H 5300 4850 50  0000 C CNN
+F 1 "STM32F302K8Ux" H 6200 4850 50  0000 C CNN
 F 2 "Package_DFN_QFN:QFN-32-1EP_5x5mm_P0.5mm_EP3.45x3.45mm" H 5250 3100 50  0001 R CNN
 F 3 "http://www.st.com/st-web-ui/static/active/en/resource/technical/document/datasheet/DM00093333.pdf" H 5750 4000 50  0001 C CNN
@@
 U 1 1 5BA7B766
 P 8450 2600
-F 0 "U?" H 8500 3278 50  0000 C CNN
-F 1 "LIS2HH12" H 8500 3187 50  0000 C CNN
+F 0 "U?" H 8200 3050 50  0000 C CNN
+F 1 "LIS2HH12" H 8750 3050 50  0000 C CNN
 F 2 "Package_LGA:LGA-12_2x2mm_P0.5mm" H 8600 3150 50  0001 L CNN
 F 3 "www.st.com/resource/en/datasheet/lis2hh12.pdf" H 8100 2600 50  0001 C CNN
@@
 U 1 1 5BB3944E
 P 8550 5000
-F 0 "U?" H 9191 5046 50  0000 L CNN
-F 1 "AT25DF041x-UxN-x" H 9191 4955 50  0000 L CNN
+F 0 "U?" H 8100 5400 50  0000 L CNN
+F 1 "AT25DF041x-UxN-x" H 8600 5400 50  0000 L CNN
 F 2 "Package_CSP:WLCSP-8_1.58x1.63x0.35mm_Layout3x5_P0.35x0.4mm_Ball0.25mm_Pad0.25mm_NSMD" H 8350 4400 50  0001 C CNN
 F 3 "http://www.adestotech.com/wp-content/uploads/DS-AT25DF041B_040.pdf" H 8550 5700 50  0001 C CNN
@@
 L Device:CP C?
 U 1 1 5BB39F29
-P 3000 1700
-F 0 "C?" H 3118 1746 50  0000 L CNN
-F 1 "CP" H 3118 1655 50  0000 L CNN
-F 2 "" H 3038 1550 50  0001 C CNN
-F 3 "~" H 3000 1700 50  0001 C CNN
-	1    3000 1700
-	1    0    0    -1
-$EndComp
-Text Notes 10100 850  0    50   ~ 0
-TODO:\n- Add ideal diode part\n- Add battery holder\n- Remove net tie
+P 2700 1700
+F 0 "C?" H 2818 1746 50  0000 L CNN
+F 1 "CP" H 2818 1655 50  0000 L CNN
+F 2 "" H 2738 1550 50  0001 C CNN
+F 3 "~" H 2700 1700 50  0001 C CNN
+	1    2700 1700
+	1    0    0    -1
+$EndComp
+Text Notes 10100 1050 0    50   ~ 0
+TODO:\n- Add ideal diode part\n- Add battery holder\n- Remove net tie\n- Add TVS array part\n- Add LED part
+$Comp
+L power:GND #PWR?
+U 1 1 5BC6AA2B
+P 8450 3250
+F 0 "#PWR?" H 8450 3000 50  0001 C CNN
+F 1 "GND" H 8455 3077 50  0000 C CNN
+F 2 "" H 8450 3250 50  0001 C CNN
+F 3 "" H 8450 3250 50  0001 C CNN
+	1    8450 3250
+	1    0    0    -1
+$EndComp
+Wire Wire Line
+	8350 3100 8350 3200
+Wire Wire Line
+	8350 3200 8450 3200
+Wire Wire Line
+	8450 3200 8450 3100
+Wire Wire Line
+	8450 3250 8450 3200
+Connection ~ 8450 3200
+Wire Wire Line
+	8550 3100 8550 3200
+Wire Wire Line
+	8550 3200 8450 3200
+$Comp
+L power:GND #PWR?
+U 1 1 5BC6B1A7
+P 8550 5550
+F 0 "#PWR?" H 8550 5300 50  0001 C CNN
+F 1 "GND" H 8555 5377 50  0000 C CNN
+F 2 "" H 8550 5550 50  0001 C CNN
+F 3 "" H 8550 5550 50  0001 C CNN
+	1    8550 5550
+	1    0    0    -1
+$EndComp
+Wire Wire Line
+	8550 5550 8550 5500
+$Comp
+L power:GND #PWR?
+U 1 1 5BC6B400
+P 1350 4500
+F 0 "#PWR?" H 1350 4250 50  0001 C CNN
+F 1 "GND" H 1355 4327 50  0000 C CNN
+F 2 "" H 1350 4500 50  0001 C CNN
+F 3 "" H 1350 4500 50  0001 C CNN
+	1    1350 4500
+	1    0    0    -1
+$EndComp
+Wire Wire Line
+	1350 4500 1350 4450
+Wire Wire Line
+	1350 4450 1250 4450
+Wire Wire Line
+	1250 4450 1250 4350
+Connection ~ 1350 4450
+Wire Wire Line
+	1350 4450 1350 4350
+$Comp
+L Regulator_Linear:TLV71333PDBV U?
+U 1 1 5BC6BDAE
+P 2350 3050
+F 0 "U?" H 2350 3392 50  0000 C CNN
+F 1 "TLV71333PDBV" H 2350 3301 50  0000 C CNN
+F 2 "Package_TO_SOT_SMD:SOT-23-5" H 2350 3350 50  0001 C CIN
+F 3 "http://www.ti.com/lit/ds/symlink/tlv713p.pdf" H 2350 3050 50  0001 C CNN
+	1    2350 3050
+	1    0    0    -1
+$EndComp
+Wire Wire Line
+	2050 3050 1950 3050
+Wire Wire Line
+	1950 3050 1950 2950
+Wire Wire Line
+	1950 2950 2050 2950
+Wire Wire Line
+	1950 2950 1750 2950
+Connection ~ 1950 2950
+$Comp
+L power:GND #PWR?
+U 1 1 5BC6CB73
+P 2350 3450
+F 0 "#PWR?" H 2350 3200 50  0001 C CNN
+F 1 "GND" H 2355 3277 50  0000 C CNN
+F 2 "" H 2350 3450 50  0001 C CNN
+F 3 "" H 2350 3450 50  0001 C CNN
+	1    2350 3450
+	1    0    0    -1
+$EndComp
+Wire Wire Line
+	2350 3450 2350 3350
+Wire Wire Line
+	1750 2950 1750 3750
+Wire Wire Line
+	1750 3750 1650 3750
 $EndSCHEMATC

Commit message: Initial PCB placement, work on schematic.
Parts:
- removed NT?: Net-Tie_2, symbol Device:Net-Tie_2
- added C102, C103: C_Small, Capacitor_SMD:C_0402_1005Metric, symbol Device:C_Small
- added C104, C105, C106, C107, C108, C109: 0.1uF, Capacitor_SMD:C_0402_1005Metric, symbol Device:C_Small
- added FID101, FID102, FID103: TestPoint, Fiducial:Fiducial_0.5mm_Dia_1mm_Outer, symbol Connector:TestPoint
- added LOGO101: Logo_Open_Hardware_Small, Symbol:OSHW-Symbol_6.7x6mm_SilkScreen, symbol Graphic:Logo_Open_Hardware_Small
- added R101: 0R-DNU, Resistor_SMD:R_0402_1005Metric, symbol Device:R_Small
- added R102: 0R, Resistor_SMD:R_0402_1005Metric, symbol Device:R_Small
- added TP101, TP102, TP103, TP104, TP105, TP106: TestPoint, TestPoint:TestPoint_Pad_D1.5mm, symbol Connector:TestPoint
- added Y101: 8MHz, Crystal:Crystal_SMD_5032-2Pin_5.0x3.2mm, symbol Device:Crystal
- J101: renamed from J?; footprint (none) -> Connector_USB:USB_Micro-B_Molex-105017-0001
- gave numbers to parts that had none: 7
Connections:
- net labels added: DEBUG0, MCU_RST, SWCLK, SWDIO, USB_DM, USB_DP, VBUS, VCC
- net labels removed: GNDA
- wire segments 31 -> 76
Other:
- note added: "TODO:\n- Add ideal diode part\n- Add battery holder\n- Remove net tie\n- Add TVS array part\n- Add LED part\n- Mftr-specific atomic xtal symbol?\n- xtal footprint\n- OSHW soldermask?"
- note removed: "TODO:\n- Add ideal diode part\n- Add battery holder\n- Remove net tie\n- Add TVS array part\n- Add LED part"

Commit message: Work on schematic
Parts:
- removed Y101: 8MHz, Crystal:Crystal_SMD_5032-2Pin_5.0x3.2mm, symbol Device:Crystal
- added C?: 47nF-C0G/NP0, Capacitor_SMD:C_0402_1005Metric, symbol Device:C_Small
- added C?: 1uF-C0G/NP0, Capacitor_SMD:C_0402_1005Metric, symbol Device:C_Small
- added C?: 4.7uF, Capacitor_SMD:C_0402_1005Metric, symbol Device:C_Small
- added R? (x2): 1k, Resistor_SMD:R_0402_1005Metric, symbol Device:R_Small
- added R?: 10R, Resistor_SMD:R_0402_1005Metric, symbol Device:R_Small
- added Y101: Crystal_GND24, Crystal:Crystal_SMD_3225-4Pin_3.2x2.5mm, symbol Device:Crystal_GND24
Connections:
- net labels added: ACCEL_SCL, ACCEL_SDA, CS_SHIELD, CS_TOUCH, SHIELD, TOUCH
- wire segments 76 -> 129
- no-connect marks 0 -> 4
Other:
- note added: "TODO:\n- Add ideal diode part\n- Add battery holder\n- Add LED part"
- note removed: "TODO:\n- Add ideal diode part\n- Add battery holder\n- Remove net tie\n- Add TVS array part\n- Add LED part\n- Mftr-specific atomic xtal symbol?\n- xtal footprint\n- OSHW soldermask?"
